Commit message: changed colors of links for rviz

File: ar3_description/urdf/ar3_macro.urdf.xacro (robot description, xacro)
@@ -2,6 +2,34 @@
 <robot xmlns:xacro="http://ros.org/wiki/xacro">
   <xacro:macro name="ar3_macro">
+    <!-- Init colour -->
+    <material name="black">
+      <color rgba="0.0 0.0 0.0 1.0"/>
+    </material>
+    <material name="dark">
+      <color rgba="0.3 0.3 0.3 1.0"/>
+    </material>
+    <material name="light_black">
+      <color rgba="0.4 0.4 0.4 1.0"/>
+    </material>
+    <material name="blue">
+      <color rgba="0.0 0.0 0.8 1.0"/>
+    </material>
+    <material name="green">
+      <color rgba="0.0 0.8 0.0 1.0"/>
+    </material>
+    <material name="grey">
+      <color rgba="0.5 0.5 0.5 1.0"/>
+    </material>
     <material name="orange">
-      <color rgba="1.0 1.0 0.0 1.0"/>
+      <color rgba="${255/255} ${108/255} ${10/255} 1.0"/>
+    </material>
+    <material name="brown">
+      <color rgba="${222/255} ${207/255} ${195/255} 1.0"/>
+    </material>
+    <material name="red">
+      <color rgba="0.8 0.0 0.0 1.0"/>
+    </material>
+    <material name="white">
+      <color rgba="1.0 1.0 1.0 1.0"/>
     </material>
     <link name="ar3_link0">
@@ -39,5 +67,5 @@
           <mesh filename="package://ar3_description/meshes/link_1.STL" />
         </geometry>
-        <material name="orange"/>
+        <material name="blue"/>
       </visual>
       <collision>
@@ -66,5 +94,5 @@
           <mesh filename="package://ar3_description/meshes/link_2.STL" />
         </geometry>
-        <material name="orange"/>
+        <material name="green"/>
       </visual>
       <collision>
@@ -93,5 +121,5 @@
           <mesh filename="package://ar3_description/meshes/link_3.STL" />
         </geometry>
-        <material name="orange"/>
+        <material name="red"/>
       </visual>
       <collision>
@@ -120,5 +148,5 @@
           <mesh filename="package://ar3_description/meshes/link_4.STL" />
         </geometry>
-        <material name="orange"/>
+        <material name="blue"/>
       </visual>
       <collision>
@@ -147,5 +175,5 @@
           <mesh filename="package://ar3_description/meshes/link_5.STL" />
         </geometry>
-        <material name="orange"/>
+        <material name="green"/>
       </visual>
       <collision>

Commit message: mostly working moveit integration

File: ar3_description/urdf/ar3_macro.urdf.xacro (robot description, xacro)
@@ -1,36 +1,6 @@
 <?xml version="1.0" ?>
 <robot xmlns:xacro="http://ros.org/wiki/xacro">
+  <xacro:include filename="$(find ar3_description)/urdf/colors.urdf.xacro" />
   <xacro:macro name="ar3_macro">
-    <!-- Init colour -->
-    <material name="black">
-      <color rgba="0.0 0.0 0.0 1.0"/>
-    </material>
-    <material name="dark">
-      <color rgba="0.3 0.3 0.3 1.0"/>
-    </material>
-    <material name="light_black">
-      <color rgba="0.4 0.4 0.4 1.0"/>
-    </material>
-    <material name="blue">
-      <color rgba="0.0 0.0 0.8 1.0"/>
-    </material>
-    <material name="green">
-      <color rgba="0.0 0.8 0.0 1.0"/>
-    </material>
-    <material name="grey">
-      <color rgba="0.5 0.5 0.5 1.0"/>
-    </material>
-    <material name="orange">
-      <color rgba="${255/255} ${108/255} ${10/255} 1.0"/>
-    </material>
-    <material name="brown">
-      <color rgba="${222/255} ${207/255} ${195/255} 1.0"/>
-    </material>
-    <material name="red">
-      <color rgba="0.8 0.0 0.0 1.0"/>
-    </material>
-    <material name="white">
-      <color rgba="1.0 1.0 1.0 1.0"/>
-    </material>
     <link name="ar3_link0">
       <!-- KDL does not support a root link with an inertia -->

File: ar3_moveit_config/config/ar3_arm.srdf.xacro (robot description, xacro)
@@ -4,6 +4,6 @@
     A URDF file must exist for this robot as well, where the joints and the links that are referenced are defined
 -->
-<robot xmlns:xacro="http://www.ros.org/wiki/xacro" name="panda">
-  <xacro:include filename="$(find moveit_resources_panda_moveit_config)/config/panda_arm.xacro" />
-  <xacro:panda_arm />
+<robot xmlns:xacro="http://www.ros.org/wiki/xacro" name="ar3">
+  <xacro:include filename="$(find ar3_moveit_config)/config/ar3_arm.xacro" />
+  <xacro:ar3_arm />
 </robot>
