Commit message: updating to latest example from ros2_control

File: ar3_description/ros2_control/ar3_position_only.ros2_control.xacro (robot description, xacro)
@@ -1,13 +1,27 @@
 <?xml version="1.0"?>
 <robot xmlns:xacro="http://www.ros.org/wiki/xacro">
-  <xacro:macro name="ar3_system_position_only" params="name prefix">
+  <xacro:macro name="ar3_system_position_only" params="name prefix use_sim:=^|false use_fake_hardware:=^|true fake_sensor_commands:=^|false slowdown:=2.0">
     <ros2_control name="${name}" type="system">
-      <hardware>
-        <plugin>fake_joint_driver/FakeJointDriver</plugin>
-        <!-- <param name="example_param_hw_start_duration_sec">2.0</param> -->
-        <!-- <param name="example_param_hw_stop_duration_sec">3.0</param> -->
-        <!-- <param name="example_param_hw_slowdown">2.0</param> -->
-      </hardware>
-      <joint name="ar3_joint1">
+      <xacro:if value="$(arg use_sim)">
+        <hardware>
+          <plugin>gazebo_ros2_control/GazeboSystem</plugin>
+        </hardware>
+      </xacro:if>
+      <xacro:unless value="$(arg use_sim)">
+        <hardware>
+          <xacro:if value="${use_fake_hardware}">
+            <plugin>fake_components/GenericSystem</plugin>
+            <param name="fake_sensor_commands">${fake_sensor_commands}</param>
+            <param name="state_following_offset">0.0</param>
+          </xacro:if>
+          <xacro:unless value="${use_fake_hardware}">
+            <plugin>ar3_hardware/AR3SystemPositionOnlyHardware</plugin>
+            <param name="example_param_hw_start_duration_sec">0.0</param>
+            <param name="example_param_hw_stop_duration_sec">3.0</param>
+            <param name="example_param_hw_slowdown">${slowdown}</param>
+          </xacro:unless>
+        </hardware>
+      </xacro:unless>
+      <joint name="${prefix}joint1">
         <command_interface name="position">
           <param name="min">-1</param>
@@ -15,7 +29,6 @@
         </command_interface>
         <state_interface name="position"/>
-        <param name="start_position">0.0</param>
       </joint>
-      <joint name="ar3_joint2">
+      <joint name="${prefix}joint2">
         <command_interface name="position">
           <param name="min">-1</param>
@@ -23,7 +36,6 @@
         </command_interface>
         <state_interface name="position"/>
-        <param name="start_position">-0.785</param>
       </joint>
-      <joint name="ar3_joint3">
+      <joint name="${prefix}joint3">
         <command_interface name="position">
           <param name="min">-1</param>
@@ -31,7 +43,6 @@
         </command_interface>
         <state_interface name="position"/>
-        <param name="start_position">0.0</param>
       </joint>
-      <joint name="ar3_joint4">
+      <joint name="${prefix}joint4">
         <command_interface name="position">
           <param name="min">-1</param>
@@ -39,7 +50,6 @@
         </command_interface>
         <state_interface name="position"/>
-        <param name="start_position">-2.356</param>
       </joint>
-      <joint name="ar3_joint5">
+      <joint name="${prefix}joint5">
         <command_interface name="position">
           <param name="min">-1</param>
@@ -47,7 +57,6 @@
         </command_interface>
         <state_interface name="position"/>
-        <param name="start_position">1.571</param>
       </joint>
-      <joint name="ar3_joint6">
+      <joint name="${prefix}joint6">
         <command_interface name="position">
           <param name="min">-1</param>
@@ -55,5 +64,4 @@
         </command_interface>
         <state_interface name="position"/>
-        <param name="start_position">0.785</param>
       </joint>
     </ros2_control>

File: ar3_description/urdf/ar3.urdf.xacro (robot description, xacro)
@@ -1,10 +1,22 @@
 <?xml version="1.0" ?>
-<robot name="ar3" xmlns:xacro="http://ros.org/wiki/xacro">
-  <!-- include common xacro files -->
-  <xacro:include filename="$(find ar3_description)/urdf/ar3_macro.urdf.xacro" />
-  <xacro:include filename="$(find ar3_description)/urdf/ar3_position_only.ros2_control.xacro" />
+<robot xmlns:xacro="http://ros.org/wiki/xacro" name="ar3_robot">
+  <xacro:arg name="prefix" default="" />
+  <!-- include AR3 macro -->
+  <xacro:include filename="$(find ar3_description)/urdf/ar3_description.urdf.xacro" />
+  <!-- include materials / colors -->
+  <xacro:include filename="$(find ar3_description)/gazebo/ar3.materials.xacro" />
+  <!-- include AR3 ros2_control description -->
+  <xacro:include filename="$(find ar3_description)/ros2_control/ar3.ros2_control.xacro" />
+  <!-- Used for fixing robot -->
+  <link name="world"/>
+  <gazebo reference="world">
+    <static>true</static>
+  </gazebo>
   <!-- Instantiate AR3 robot. Call this xacro macro in your own urdf.xacro to
        attach accessories to the AR3. -->
-  <xacro:ar3_macro/>
-  <xacro:ar3_system_position_only name="ar3_position_only" prefix=""/>
+  <xacro:ar3 parent="world" prefix="$(arg prefix)">
+    <origin xyz="0 0 0" rpy="0 0 0" />
+  </xacro:ar3>
+  <xacro:ar3_ros2_control
+      name="ar3" prefix="$(arg prefix)"/>
 </robot>

File: ar3_description/urdf/ar3_description.urdf.xacro (robot description, xacro)
@@ -1,14 +1,11 @@
 <?xml version="1.0" ?>
 <robot xmlns:xacro="http://ros.org/wiki/xacro">
-  <xacro:include filename="$(find ar3_description)/urdf/colors.urdf.xacro" />
-  <xacro:macro name="ar3_macro">
-    <link name="ar3_link0">
-      <!-- KDL does not support a root link with an inertia -->
-      <!-- <inertial> -->
-      <!--   <origin xyz="-4.6941E-06 0.054174 0.038824" rpy="0 0 0" /> -->
-      <!--   <mass value="0.7102" />        -->
-      <!--   <inertia ixx="0.0039943" ixy="3.697E-07" ixz="-5.7364E-08" -->
-      <!--            iyy="0.0014946" iyz="-0.00036051" izz="0.0042554" /> -->
-      <!-- </inertial> -->
+  <xacro:macro name="ar3" params="parent prefix *origin">
+    <joint name="${prefix}base_joint" type="fixed">
+      <xacro:insert_block name="origin" />
+      <parent link="${parent}"/>
+      <child link="${prefix}base_link" />
+    </joint>
+    <link name="${prefix}base_link">
       <visual>
         <origin xyz="0 0 0" rpy="0 0 0" />
@@ -25,5 +22,5 @@
       </collision>
     </link>
-    <link name="ar3_link1">
+    <link name="${prefix}link1">
       <inertial>
         <origin xyz="-0.022706 0.04294 -0.12205" rpy="0 0 0" />
@@ -46,11 +43,11 @@
       </collision>
     </link>
-    <joint name="ar3_joint1" type="continuous">
+    <joint name="${prefix}joint1" type="continuous">
       <origin xyz="0 0 0.003445" rpy="3.1416 -1.0248E-21 -1.6736E-05" />
-      <parent link="ar3_link0" />
-      <child link="ar3_link1" />
+      <parent link="${prefix}base_link" />
+      <child link="${prefix}link1" />
       <axis xyz="0 0 1" />
     </joint>
-    <link name="ar3_link2">
+    <link name="${prefix}link2">
       <inertial>
         <origin xyz="0.064818 -0.11189 -0.038671" rpy="0 0 0" />
@@ -73,11 +70,11 @@
       </collision>
     </link>
-    <joint name="ar3_joint2" type="continuous">
+    <joint name="${prefix}joint2" type="continuous">
       <origin xyz="0 0.064146 -0.16608" rpy="1.5708 0.5236 -1.5708" />
-      <parent link="ar3_link1" />
-      <child link="ar3_link2" />
+      <parent link="${prefix}link1" />
+      <child link="${prefix}link2" />
       <axis xyz="0 0 1" />
     </joint>
-    <link name="ar3_link3">
+    <link name="${prefix}link3">
       <inertial>
         <origin xyz="-0.00029765 -0.023661 -0.0019125" rpy="0 0 0" />
@@ -100,11 +97,11 @@
       </collision>
     </link>
-    <joint name="ar3_joint3" type="continuous">
+    <joint name="${prefix}joint3" type="continuous">
       <origin xyz="0.1525 -0.26414 0" rpy="3.3431E-16 -1.4164E-16 -2.618" />
-      <parent link="ar3_link2" />
-      <child link="ar3_link3" />
+      <parent link="${prefix}link2" />
+      <child link="${prefix}link3" />
       <axis xyz="0 0 -1" />
     </joint>
-    <link name="ar3_link4">
+    <link name="${prefix}link4">
       <inertial>
         <origin xyz="-0.0016798 -0.00057319 -0.074404" rpy="0 0 0" />
@@ -127,11 +124,11 @@
       </collision>
     </link>
-    <joint name="ar3_joint4" type="continuous">
+    <joint name="${prefix}joint4" type="continuous">
       <origin xyz="0 0 0.00675" rpy="1.5708 -1.2554 -1.5708" />
-      <parent link="ar3_link3" />
-      <child link="ar3_link4" />
+      <parent link="${prefix}link3" />
+      <child link="${prefix}link4" />
       <axis xyz="0 0 -1" />
     </joint>
-    <link name="ar3_link5">
+    <link name="${prefix}link5">
       <inertial>
         <origin xyz="0.0015066 -1.3102E-05 -0.012585" rpy="0 0 0" />
@@ -154,11 +151,11 @@
       </collision>
     </link>
-    <joint name="ar3_joint5" type="continuous">
+    <joint name="${prefix}joint5" type="continuous">
       <origin xyz="0 0 -0.22225" rpy="3.1416 0 -2.8262" />
-      <parent link="ar3_link4" />
-      <child link="ar3_link5" />
+      <parent link="${prefix}link4" />
+      <child link="${prefix}link5" />
       <axis xyz="-1 0 0" />
     </joint>
-    <link name="ar3_link6">
+    <link name="${prefix}link6">
       <inertial>
         <origin xyz="2.9287E-10 -1.6472E-09 0.0091432" rpy="0 0 0" />
@@ -181,8 +178,8 @@
       </collision>
     </link>
-    <joint name="ar3_joint6" type="continuous">
+    <joint name="${prefix}joint6" type="continuous">
       <origin xyz="-0.000294 0 0.02117" rpy="0 0 3.1416" />
-      <parent link="ar3_link5" />
-      <child link="ar3_link6" />
+      <parent link="${prefix}link5" />
+      <child link="${prefix}link6" />
       <axis xyz="0 0 -1" />
     </joint>
