Commit message: added firmware version to arduino, using TimeoutSerial for comms

File: ar3_description/ros2_control/ar3.ros2_control.xacro (robot description, xacro)
@@ -1,5 +1,5 @@
 <?xml version="1.0"?>
 <robot xmlns:xacro="http://www.ros.org/wiki/xacro">
-  <xacro:macro name="ar3_ros2_control" params="name prefix">
+  <xacro:macro name="ar3_ros2_control" params="name prefix serial_device serial_baudrate firmware_version">
     <ros2_control name="${name}" type="system">
       <hardware>
@@ -8,4 +8,7 @@
         <param name="example_param_hw_stop_duration_sec">3.0</param>
         <param name="example_param_hw_slowdown">100</param>
+        <param name="serial_device">${serial_device}</param>
+        <param name="serial_baudrate">${serial_baudrate}</param>
+        <param name="firmware_version">${firmware_version}</param>
       </hardware>
       <joint name="${prefix}joint1">

File: ar3_description/urdf/ar3.urdf.xacro (robot description, xacro)
@@ -2,4 +2,7 @@
 <robot xmlns:xacro="http://ros.org/wiki/xacro" name="ar3_robot">
   <xacro:arg name="prefix" default="" />
+  <xacro:arg name="serial_device" default="" />
+  <xacro:arg name="serial_baudrate" default="" />
+  <xacro:arg name="firmware_version" default="" />
   <!-- include AR3 macro -->
   <xacro:include filename="$(find ar3_description)/urdf/ar3_description.urdf.xacro" />
@@ -19,4 +22,4 @@
   </xacro:ar3>
   <xacro:ar3_ros2_control
-      name="ar3" prefix="$(arg prefix)"/>
+      name="ar3" prefix="$(arg prefix)" serial_device="$(arg serial_device)" serial_baudrate="$(arg serial_baudrate)" firmware_version="$(arg firmware_version)"/>
 </robot>
