Commit message: figuring our encoder logic

File: ar3_description/ros2_control/ar3_system_position_only.ros2_control.xacro (robot description, xacro)
@@ -1,5 +1,5 @@
 <?xml version="1.0"?>
 <robot xmlns:xacro="http://www.ros.org/wiki/xacro">
-  <xacro:macro name="ar3_system_position_only" params="name prefix use_sim:=^|false use_fake_hardware:=^|true fake_sensor_commands:=^|false slowdown:=2.0">
+  <xacro:macro name="ar3_system_position_only" params="name prefix serial_device serial_baudrate firmware_version use_sim:=^|false use_fake_hardware:=^|true fake_sensor_commands:=^|false">
     <ros2_control name="${name}" type="system">
       <xacro:if value="$(arg use_sim)">
@@ -17,7 +17,7 @@
           <xacro:unless value="${use_fake_hardware}">
             <plugin>ar3_hardware/AR3SystemPositionOnlyHardware</plugin>
-            <param name="example_param_hw_start_duration_sec">0.0</param>
-            <param name="example_param_hw_stop_duration_sec">3.0</param>
-            <param name="example_param_hw_slowdown">${slowdown}</param>
+            <param name="serial_device">${serial_device}</param>
+            <param name="serial_baudrate">${serial_baudrate}</param>
+            <param name="firmware_version">${firmware_version}</param>
           </xacro:unless>
         </hardware>

File: ar3_description/urdf/ar3.urdf.xacro (robot description, xacro)
@@ -2,7 +2,12 @@
 <robot xmlns:xacro="http://ros.org/wiki/xacro" name="ar3_robot">
   <xacro:arg name="prefix" default="" />
+  <!-- Serial hardware arguments -->
   <xacro:arg name="serial_device" default="" />
   <xacro:arg name="serial_baudrate" default="" />
   <xacro:arg name="firmware_version" default="" />
+  <!-- Simulation arguments -->
+  <xacro:arg name="use_sim" default="false" />
+  <xacro:arg name="use_fake_hardware" default="false"/>
+  <xacro:arg name="fake_sensor_commands" default="false"/>
   <!-- include AR3 macro -->
   <xacro:include filename="$(find ar3_description)/urdf/ar3_description.urdf.xacro" />
@@ -10,5 +15,6 @@
   <xacro:include filename="$(find ar3_description)/gazebo/ar3.materials.xacro" />
   <!-- include AR3 ros2_control description -->
-  <xacro:include filename="$(find ar3_description)/ros2_control/ar3.ros2_control.xacro" />
+  <!-- <xacro:include filename="$(find ar3_description)/ros2_control/ar3.ros2_control.xacro" /> -->
+  <xacro:include filename="$(find ar3_description)/ros2_control/ar3_system_position_only.ros2_control.xacro" />
   <!-- Used for fixing robot -->
   <link name="world"/>
@@ -21,5 +27,15 @@
     <origin xyz="0 0 0" rpy="0 0 0" />
   </xacro:ar3>
-  <xacro:ar3_ros2_control
-      name="ar3" prefix="$(arg prefix)" serial_device="$(arg serial_device)" serial_baudrate="$(arg serial_baudrate)" firmware_version="$(arg firmware_version)"/>
+  <!-- <xacro:ar3_ros2_control -->
+  <!--     name="ar3" prefix="$(arg prefix)" serial_device="$(arg serial_device)" serial_baudrate="$(arg serial_baudrate)" firmware_version="$(arg firmware_version)"/> -->
+  <xacro:ar3_system_position_only
+      name="ar3"
+      prefix="$(arg prefix)"
+      serial_device="$(arg serial_device)"
+      serial_baudrate="$(arg serial_baudrate)"
+      firmware_version="$(arg firmware_version)"
+      use_sim="$(arg use_sim)"
+      use_fake_hardware="$(arg use_fake_hardware)"
+      fake_sensor_commands="$(arg fake_sensor_commands)"
+      />
 </robot>

Commit message: using sim_gazebo instead of use_sim

File: ar3_description/ros2_control/ar3_system_position_only.ros2_control.xacro (robot description, xacro)
@@ -1,12 +1,12 @@
 <?xml version="1.0"?>
 <robot xmlns:xacro="http://www.ros.org/wiki/xacro">
-  <xacro:macro name="ar3_system_position_only" params="name prefix serial_device serial_baudrate firmware_version use_sim:=^|false use_fake_hardware:=^|true fake_sensor_commands:=^|false">
+  <xacro:macro name="ar3_system_position_only" params="name prefix serial_device serial_baudrate firmware_version sim_gazebo:=^|false use_fake_hardware:=^|true fake_sensor_commands:=^|false">
     <ros2_control name="${name}" type="system">
-      <xacro:if value="$(arg use_sim)">
+      <xacro:if value="$(arg sim_gazebo)">
         <hardware>
           <plugin>gazebo_ros2_control/GazeboSystem</plugin>
         </hardware>
       </xacro:if>
-      <xacro:unless value="$(arg use_sim)">
+      <xacro:unless value="$(arg sim_gazebo)">
         <hardware>
           <xacro:if value="${use_fake_hardware}">
