Commit message: first working control of AR3 robot arm with moveit2

File: ar3_moveit_config/config/ar3_arm.srdf.xacro (robot description, xacro)
@@ -4,5 +4,5 @@
     A URDF file must exist for this robot as well, where the joints and the links that are referenced are defined
 -->
-<robot xmlns:xacro="http://www.ros.org/wiki/xacro" name="ar3">
+<robot xmlns:xacro="http://www.ros.org/wiki/xacro" name="ar3_robot">
   <xacro:include filename="$(find ar3_moveit_config)/config/ar3_arm.xacro" />
   <xacro:ar3_arm />

File: ar3_moveit_config/config/ar3_arm.xacro (robot description, xacro)
@@ -1,4 +1,4 @@
 <?xml version="1.0" ?>
-<robot xmlns:xacro="http://www.ros.org/wiki/xacro" name="ar3">
+<robot xmlns:xacro="http://www.ros.org/wiki/xacro" name="ar3_robot">
   <xacro:macro name="ar3_arm">
     <!--GROUPS - Representation of a set of joints and links. This can be useful for specifying DOF to plan for, defining arms, end effectors, etc-->
@@ -8,51 +8,51 @@
     <!--SUBGROUPS - Groups can also be formed by referencing to already defined group names-->
     <group name="ar3_arm">
-      <chain base_link="ar3_link0" tip_link="ar3_link6" />
+      <chain base_link="base_link" tip_link="link6" />
     </group>
     <!--GROUP STATES - Purpose - Define a named state for a particular group, in terms of joint values. This is useful to define states like 'folded arms'-->
-    <group_state name="ready" group="ar3_arm">
-      <joint name="ar3_joint1" value="0" />
-      <joint name="ar3_joint2" value="-0.785" />
-      <joint name="ar3_joint3" value="0" />
-      <joint name="ar3_joint4" value="-2.356" />
-      <joint name="ar3_joint5" value="0" />
-      <joint name="ar3_joint6" value="1.571" />
+    <group_state name="home" group="ar3_arm">
+      <joint name="joint1" value="0" />
+      <joint name="joint2" value="-1.6" />
+      <joint name="joint3" value="0.05" />
+      <joint name="joint4" value="0.0" />
+      <joint name="joint5" value="0.6" />
+      <joint name="joint6" value="0.0" />
     </group_state>
     <group_state name="extended" group="ar3_arm">
-      <joint name="ar3_joint1" value="0" />
-      <joint name="ar3_joint2" value="0" />
-      <joint name="ar3_joint3" value="0" />
-      <joint name="ar3_joint4" value="0" />
-      <joint name="ar3_joint5" value="0" />
-      <joint name="ar3_joint6" value="1.571" />
+      <joint name="joint1" value="0" />
+      <joint name="joint2" value="0" />
+      <joint name="joint3" value="0" />
+      <joint name="joint4" value="0" />
+      <joint name="joint5" value="0" />
+      <joint name="joint6" value="1.571" />
     </group_state>
-    <group_state name="transport" group="ar3_arm">
-      <joint name="ar3_joint1" value="0" />
-      <joint name="ar3_joint2" value="-0.5599" />
-      <joint name="ar3_joint3" value="0" />
-      <joint name="ar3_joint4" value="-2.97" />
-      <joint name="ar3_joint5" value="0" />
-      <joint name="ar3_joint6" value="0" />
+    <group_state name="shutdown" group="ar3_arm">
+      <joint name="joint1" value="0" />
+      <joint name="joint2" value="-1.5" />
+      <joint name="joint3" value="1.45" />
+      <joint name="joint4" value="0" />
+      <joint name="joint5" value="-0.6" />
+      <joint name="joint6" value="0" />
     </group_state>
     <!--END EFFECTOR - Purpose - Represent information about an end effector.-->
     <!--VIRTUAL JOINT - Purpose - this element defines a virtual joint between a robot link and an external frame of reference (considered fixed with respect to the robot)-->
-    <virtual_joint name="virtual_joint" type="floating" parent_frame="world" child_link="ar3_link0" />
+    <virtual_joint name="virtual_joint" type="floating" parent_frame="world" child_link="base_link" />
     <!--DISABLE COLLISIONS - By default it is assumed that any link of the robot could potentially come into collision with any other link in the robot. This tag disables collision checking between a specified pair of links. -->
-    <disable_collisions link1="ar3_link0" link2="ar3_link1" reason="Adjacent" />
-    <disable_collisions link1="ar3_link0" link2="ar3_link2" reason="Never" />
-    <disable_collisions link1="ar3_link0" link2="ar3_link3" reason="Never" />
-    <disable_collisions link1="ar3_link0" link2="ar3_link4" reason="Never" />
-    <disable_collisions link1="ar3_link1" link2="ar3_link2" reason="Adjacent" />
-    <disable_collisions link1="ar3_link1" link2="ar3_link3" reason="Never" />
-    <disable_collisions link1="ar3_link1" link2="ar3_link4" reason="Never" />
-    <disable_collisions link1="ar3_link2" link2="ar3_link3" reason="Adjacent" />
-    <disable_collisions link1="ar3_link2" link2="ar3_link4" reason="Never" />
-    <disable_collisions link1="ar3_link2" link2="ar3_link6" reason="Never" />
-    <disable_collisions link1="ar3_link3" link2="ar3_link4" reason="Adjacent" />
-    <disable_collisions link1="ar3_link3" link2="ar3_link5" reason="Never" />
-    <disable_collisions link1="ar3_link3" link2="ar3_link6" reason="Never" />
-    <disable_collisions link1="ar3_link4" link2="ar3_link5" reason="Adjacent" />
-    <disable_collisions link1="ar3_link4" link2="ar3_link6" reason="Never" />
-    <disable_collisions link1="ar3_link5" link2="ar3_link6" reason="Adjacent" />
+    <disable_collisions link1="base_link" link2="link1" reason="Adjacent" />
+    <disable_collisions link1="base_link" link2="link2" reason="Never" />
+    <disable_collisions link1="base_link" link2="link3" reason="Never" />
+    <disable_collisions link1="base_link" link2="link4" reason="Never" />
+    <disable_collisions link1="link1" link2="link2" reason="Adjacent" />
+    <disable_collisions link1="link1" link2="link3" reason="Never" />
+    <disable_collisions link1="link1" link2="link4" reason="Never" />
+    <disable_collisions link1="link2" link2="link3" reason="Adjacent" />
+    <disable_collisions link1="link2" link2="link4" reason="Never" />
+    <disable_collisions link1="link2" link2="link6" reason="Never" />
+    <disable_collisions link1="link3" link2="link4" reason="Adjacent" />
+    <disable_collisions link1="link3" link2="link5" reason="Never" />
+    <disable_collisions link1="link3" link2="link6" reason="Never" />
+    <disable_collisions link1="link4" link2="link5" reason="Adjacent" />
+    <disable_collisions link1="link4" link2="link6" reason="Never" />
+    <disable_collisions link1="link5" link2="link6" reason="Adjacent" />
   </xacro:macro>
 </robot>
